File: pcb/choc/pcb.kicad_pcb (KiCad board)
At the start: 2 copper layers, 154.2 x 86 mm, 70 parts, among them J1 MJ-4PP-9, J2 USB_C_Receptacle_USB2.0, J3 Conn_01x04_Female, J4 Conn_01x08_Female, SW1 SW_PUSH, SW10 SW_PUSH, SW11 SW_PUSH, SW12 SW_PUSH, SW13 SW_PUSH, SW14 SW_PUSH, SW15 SW_PUSH, SW16 SW_PUSH, SW17 SW_PUSH, SW18 SW_PUSH, SW19 SW_PUSH, SW2 SW_PUSH, SW3 SW_PUSH, SW4 SW_PUSH, SW5 SW_PUSH, SW6 SW_PUSH, SW7 SW_PUSH, SW8 SW_PUSH, SW9 SW_PUSH, U1 rp2040-zero, U2 rp2040-zero, U3 roller

Commit message: draft 1
Parts:
- removed J3: Conn_01x04_Female, zzkeeb:Pointing_Cirque-adapter
- removed J4: Conn_01x08_Female, Connector_JST:JST_PH_S8B-PH-K_1x08_P2.00mm_Horizontal
- added BR1: MountingHole, zzkeeb:Hole_Breakaway-Tabs, F.Cu at (178.7, 85.9)
- added BR2: MountingHole, zzkeeb:Hole_Breakaway-Tabs, F.Cu at (178.7, 115.0)
- added BR3: MountingHole, zzkeeb:Hole_Breakaway-Tabs, F.Cu at (183.3, 86.0)
- added BR4: MountingHole, zzkeeb:Hole_Breakaway-Tabs, F.Cu at (183.3, 115.0)
- added CIRQUE1: Conn_01x12_Female, zzkeeb:Connector_FFC-FPC-vertical-12pin, F.Cu at (174.5, 113.5)
- added CIRQUE2: Conn_01x12_Female, zzkeeb:Connector_FPC-FFC-adapter-12pin, F.Cu at (164.0, 109.0)
- added CIRQUE3: Conn_01x12_Female, zzkeeb:Connector_FFC-FPC-vertical-12pin, F.Cu at (187.5, 113.5)
- added CIRQUE4: Conn_01x12_Female, zzkeeb:Connector_FPC-FFC-adapter-12pin, F.Cu at (198.0, 121.5)
- added D21: D_Small, zzkeeb:Diode_1N4148-SOD123, B.Cu at (329.2, 111.2)
- added D22: D_Small, zzkeeb:Diode_1N4148-SOD123, B.Cu at (288.5, 91.0)
- added D23: D_Small, zzkeeb:Diode_1N4148-SOD123, B.Cu at (270.5, 87.0)
- added D24: D_Small, zzkeeb:Diode_1N4148-SOD123, B.Cu at (252.3, 94.8)
- added D25: D_Small, zzkeeb:Diode_1N4148-SOD123, B.Cu at (234.5, 95.0)
- added D26: D_Small, zzkeeb:Diode_1N4148-SOD123, B.Cu at (311.0, 111.0)
- added D27: D_Small, zzkeeb:Diode_1N4148-SOD123, B.Cu at (288.5, 108.0)
- added D28: D_Small, zzkeeb:Diode_1N4148-SOD123, B.Cu at (270.0, 104.0)
- added D29: D_Small, zzkeeb:Diode_1N4148-SOD123, B.Cu at (252.5, 112.0)
- added D30: D_Small, zzkeeb:Diode_1N4148-SOD123, B.Cu at (234.5, 112.0)
- added D31: D_Small, zzkeeb:Diode_1N4148-SOD123, B.Cu at (300.5, 111.0)
- added D32: D_Small, zzkeeb:Diode_1N4148-SOD123, B.Cu at (288.5, 125.0)
- added D33: D_Small, zzkeeb:Diode_1N4148-SOD123, B.Cu at (270.5, 121.0)
- added D34: D_Small, zzkeeb:Diode_1N4148-SOD123, B.Cu at (256.3, 128.0)
- added D35: D_Small, zzkeeb:Diode_1N4148-SOD123, B.Cu at (239.0, 128.0)
- added D36: D_Small, zzkeeb:Diode_1N4148-SOD123, B.Cu at (320.0, 111.5)
- added D37: D_Small, zzkeeb:Diode_1N4148-SOD123, B.Cu at (274.5, 124.0)
- added D38: D_Small, zzkeeb:Diode_1N4148-SOD123, B.Cu at (248.5, 128.0)
- added D39: D_Small, zzkeeb:Diode_1N4148-SOD123, B.Cu at (228.0, 129.5)
- added D40: D_Small, zzkeeb:Diode_1N4148-SOD123, B.Cu at (217.5, 133.0)
- added DISP1: Conn_01x08_Female, zzkeeb:Connector_JST_PH_S8B-PH-K_1x08_P2.00mm_Horizontal, F.Cu at (152.0, 126.6)
- added DISP2: Conn_01x08_Female, zzkeeb:Connector_JST_PH_S8B-PH-K_1x08_P2.00mm_Horizontal, F.Cu at (196.0, 126.5)
- added H10: MountingHole, zzkeeb:Hole_M2-spacer, F.Cu at (195.0, 81.0)
- added H11: MountingHole, zzkeeb:Hole_M2-spacer, F.Cu at (174.5, 129.0)
- added H12: MountingHole, zzkeeb:Hole_M2-spacer, F.Cu at (265.0, 124.0)
- added H5: MountingHole, zzkeeb:Hole_M2-spacer, F.Cu at (187.5, 129.0)
- added H6: MountingHole, zzkeeb:Hole_M2-spacer, F.Cu at (141.5, 128.0)
- added H7: MountingHole, zzkeeb:Hole_M2-spacer, F.Cu at (315.5, 111.0)
- added H8: MountingHole, zzkeeb:Hole_M2-spacer, F.Cu at (243.5, 94.0)
- added H9: MountingHole, zzkeeb:Hole_M2-spacer, F.Cu at (222.5, 128.0)
- added I2C1: Conn_01x04_Female, zzkeeb:Pointing_Cirque-adapter, F.Cu at (146.5, 115.5)
- added I2C2: Conn_01x04_Female, zzkeeb:Pointing_Cirque-adapter, F.Cu at (215.5, 115.5)
- added LED20: YS-SK6812MINI-E, zzkeeb:LED_SK6812-MINI-E, F.Cu at (215.4, 138.8)
- added LED21: YS-SK6812MINI-E, zzkeeb:LED_SK6812-MINI-E, F.Cu at (235.2, 133.6)
- added LED22: YS-SK6812MINI-E, zzkeeb:LED_SK6812-MINI-E, F.Cu at (255.5, 131.8)
- added LED23: YS-SK6812MINI-E, zzkeeb:LED_SK6812-MINI-E, F.Cu at (252.5, 114.8)
- added LED24: YS-SK6812MINI-E, zzkeeb:LED_SK6812-MINI-E, F.Cu at (234.5, 114.8)
- added LED25: YS-SK6812MINI-E, zzkeeb:LED_SK6812-MINI-E, F.Cu at (234.5, 97.8)
- added LED26: YS-SK6812MINI-E, zzkeeb:LED_SK6812-MINI-E, F.Cu at (252.6, 97.8)
- added LED27: YS-SK6812MINI-E, zzkeeb:LED_SK6812-MINI-E, F.Cu at (270.5, 89.8)
- added LED28: YS-SK6812MINI-E, zzkeeb:LED_SK6812-MINI-E, F.Cu at (270.5, 106.8)
- added LED29: YS-SK6812MINI-E, zzkeeb:LED_SK6812-MINI-E, F.Cu at (288.5, 110.8)
- added LED30: YS-SK6812MINI-E, zzkeeb:LED_SK6812-MINI-E, F.Cu at (306.5, 114.8)
- added LED31: YS-SK6812MINI-E, zzkeeb:LED_SK6812-MINI-E, F.Cu at (324.6, 114.8)
- added LED32: YS-SK6812MINI-E, zzkeeb:LED_SK6812-MINI-E, F.Cu at (324.5, 97.8)
- added LED33: YS-SK6812MINI-E, zzkeeb:LED_SK6812-MINI-E, F.Cu at (306.5, 97.8)
- added LED34: YS-SK6812MINI-E, zzkeeb:LED_SK6812-MINI-E, F.Cu at (288.5, 93.8)
- added LED35: YS-SK6812MINI-E, zzkeeb:LED_SK6812-MINI-E, F.Cu at (288.5, 76.8)
- added LED36: YS-SK6812MINI-E, zzkeeb:LED_SK6812-MINI-E, F.Cu at (270.5, 72.8)
- added LED37: YS-SK6812MINI-E, zzkeeb:LED_SK6812-MINI-E, F.Cu at (252.5, 80.8)
- added LED38: YS-SK6812MINI-E, zzkeeb:LED_SK6812-MINI-E, F.Cu at (234.5, 80.8)
- added RE2: RotaryEncoder_Switch, zzkeeb:RotaryEncoder_EC11, F.Cu at (275.0, 133.5)
- added ROLL2: roller, zzkeeb:RotaryEncoder_EVQWGD001, F.Cu at (272.8, 135.3)
- added SW20: Switch, zzkeeb:Switch_ChocV1-hotswap, F.Cu at (324.5, 102.5)
- added SW21: Switch, zzkeeb:Switch_ChocV1-hotswap, F.Cu at (288.5, 81.5)
- added SW22: Switch, zzkeeb:Switch_ChocV1-hotswap, F.Cu at (270.5, 77.5)
- added SW23: Switch, zzkeeb:Switch_ChocV1-hotswap, F.Cu at (252.5, 85.5)
- added SW24: Switch, zzkeeb:Switch_ChocV1-hotswap, F.Cu at (234.5, 85.5)
- added SW25: Switch, zzkeeb:Switch_ChocV1-hotswap, F.Cu at (306.5, 102.5)
- added SW26: Switch, zzkeeb:Switch_ChocV1-hotswap, F.Cu at (288.5, 98.5)
- added SW27: Switch, zzkeeb:Switch_ChocV1-hotswap, F.Cu at (270.5, 94.5)
- added SW28: Switch, zzkeeb:Switch_ChocV1-hotswap, F.Cu at (252.5, 102.5)
- added SW29: Switch, zzkeeb:Switch_ChocV1-hotswap, F.Cu at (234.5, 102.5)
- added SW30: Switch, zzkeeb:Switch_ChocV1-hotswap, F.Cu at (306.5, 119.5)
- added SW31: Switch, zzkeeb:Switch_ChocV1-hotswap, F.Cu at (288.5, 115.5)
- added SW32: Switch, zzkeeb:Switch_ChocV1-hotswap, F.Cu at (270.5, 111.5)
- added SW33: Switch, zzkeeb:Switch_ChocV1-hotswap, F.Cu at (252.5, 119.5)
- added SW34: Switch, zzkeeb:Switch_ChocV1-hotswap, F.Cu at (234.5, 119.5)
- added SW35: Switch, zzkeeb:Switch_ChocV1-hotswap, F.Cu at (324.5, 119.5)
- added SW36: Switch, zzkeeb:Switch_ChocV1-hotswap, F.Cu at (255.5, 136.5)
- added SW37: Switch, zzkeeb:Switch_ChocV1-hotswap, F.Cu at (236.0, 138.2)
- added SW38: Switch, zzkeeb:Switch_ChocV1-hotswap, F.Cu at (217.0, 143.2)
- added TRRS2: MJ-4PP-9, zzkeeb:Connector_TRRS, F.Cu at (188.0, 76.8)
- added USB2: USB_C_Receptacle_USB2.0, zzkeeb:Connector_USB-C-mid-mount-ali-data, F.Cu at (187.8, 98.2)
- D1, D10, D11, D12, D13, D14, D15, D16, D17, D18, D19, D2, D20, D3, D4, D5, D6, D7, D8, D9: footprint zzkeeb:Diode_1N4148-SOD123-reversible -> zzkeeb:Diode_1N4148-SOD123; moved to B.Cu
- LED1, LED10, LED11, LED12, LED13, LED14, LED15, LED16, LED17, LED18, LED19, LED2, LED3, LED4, LED5, LED6, LED7, LED8, LED9: footprint zzkeeb:LED_SK6812-MINI-E-reversible -> zzkeeb:LED_SK6812-MINI-E
- MCU1: renamed from U1; footprint zzkeeb:MCU_rp2040-zero-smd -> zzkeeb:MCU_rp2040-zero-tht-pads; moved to F.Cu
- MCU2: renamed from U2; footprint zzkeeb:MCU_rp2040-zero-smd -> zzkeeb:MCU_rp2040-zero-tht-pads
- SW1, SW10, SW11, SW12, SW13, SW14, SW15, SW16, SW17, SW18, SW19, SW2, SW3, SW4, SW5, SW6, SW7, SW8, SW9: value SW_PUSH -> Switch; footprint zzkeeb:Switch_ChocV1-hotswap-reversible -> zzkeeb:Switch_ChocV1-hotswap
- TRRS1: renamed from J1; footprint zzkeeb:Connector_TRRS-reversible -> zzkeeb:Connector_TRRS
- USB1: renamed from J2; footprint zzkeeb:Connector_USB-C-mid-mount-ali-reversible-data -> zzkeeb:Connector_USB-C-mid-mount-ali-data
- moved H2 63.6 mm to (68.0, 127.0)
- moved D19 50.9 mm to (127.3, 141.2), turned to -10 degrees
- moved D20 50.5 mm to (145.6, 146.3), turned to -20 degrees
- moved D18 50.4 mm to (108.2, 139.3), turned to 0 degrees
- moved D11 49.0 mm to (57.2, 122.3), turned to 0 degrees
- moved D16 48.2 mm to (39.2, 122.3), turned to 0 degrees
- moved H1 45.8 mm to (167.0, 81.0)
- moved MCU2 45.7 mm to (211.8, 88.8)
- moved USB1 44.0 mm to (174.2, 98.2)
- moved H4 42.1 mm to (103.5, 74.0)
- moved MCU1 40.5 mm to (149.5, 88.8), turned to 0 degrees
- moved LED17 39.3 mm to (106.5, 131.8)
- moved LED18 39.3 mm to (126.8, 133.6)
- moved LED19 39.3 mm to (146.6, 138.8)
- moved LED1 39.3 mm to (127.5, 80.8)
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- renumbered U3 to ROLL1
Connections:
- MCU1 pad 10: col0 -> CS
- MCU1 pad 11: col1 -> SCLK/SDA
- MCU1 pad 12: col2 -> MOSI/SCL
- MCU1 pad 13: col3 -> MISO/DC
- MCU1 pad 14: col4 -> RST
- MCU1 pad 15: ENCA -> row3
- MCU1 pad 16: LED -> row2
- MCU1 pad 17: row0 -> row1
- MCU1 pad 18: row1 -> row0
- MCU1 pad 19: row2 -> BL
- MCU1 pad 20: row3 -> LED
- MCU1 pad 3: SCLK/SDA -> col0
- MCU1 pad 4: MOSI/SCL -> col1
- MCU1 pad 5: MISO/DC -> col2
- MCU1 pad 6: CS -> col3
- MCU1 pad 7: RST -> col4
- MCU1 pad 8: BL -> ENCA
- MCU2 pad 1: TX -> TX_r
- MCU2 pad 10: col4 -> CS_r
- MCU2 pad 11: col3 -> SCLK/SDA_r
- MCU2 pad 12: col2 -> MOSI/SCL_r
- MCU2 pad 13: col1 -> MISO/DC_r
- MCU2 pad 14: col0 -> RST_r
- MCU2 pad 15: ENCB -> row3_r
- MCU2 pad 16: LED -> row2_r
- MCU2 pad 17: row0 -> row1_r
- MCU2 pad 18: row1 -> row0_r
- MCU2 pad 19: row2 -> BL_r
- MCU2 pad 2: RX -> RX_r
- MCU2 pad 20: row3 -> LED_r
- MCU2 pad 21: VCC -> VDD
- MCU2 pad 22: GND -> GNDA
- MCU2 pad 3: SCLK/SDA -> col0_r
- MCU2 pad 4: MOSI/SCL -> col1_r
- MCU2 pad 5: MISO/DC -> col2_r
- MCU2 pad 6: CS -> col3_r
- MCU2 pad 7: RST -> col4_r
- MCU2 pad 8: BL -> ENCA_r
- MCU2 pad 9: ENCA -> ENCB_r
- TRRS1 pad A: TX -> (no net)
- TRRS1 pad B: RX -> (no net)
- TRRS1 pad C: GND -> (no net)
- TRRS1 pad D: VCC -> (no net)
Routing:
- net col0: track 224.3 -> 0.00 mm, vias 1 -> 0
- net col1: track 162.4 -> 0.00 mm, vias 1 -> 0
- net col3: track 154.0 -> 0.00 mm, vias 1 -> 0
- net VCC: track 148.9 -> 0.00 mm, vias 3 -> 0
- net col2: track 130.2 -> 0.00 mm, vias 1 -> 0
- net row3: track 106.9 -> 0.00 mm, vias 6 -> 0
- net col4: track 102.4 -> 0.00 mm, vias 1 -> 0
- net row2: track 97.5 -> 0.00 mm, vias 6 -> 0
- net MISO/DC: track 86.6 -> 0.00 mm, vias 1 -> 0
- net TX: track 85.4 -> 0.00 mm, vias 1 -> 0
- net CS: track 83.8 -> 0.00 mm, vias 1 -> 0
- net SCLK/SDA: track 82.9 -> 0.00 mm, vias 1 -> 0
- net ENCB: track 82.0 -> 0.00 mm, vias 1 -> 0
- net MOSI/SCL: track 80.7 -> 0.00 mm, vias 1 -> 0
- net row1: track 77.3 -> 0.00 mm, vias 6 -> 0
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Other:
- board size 154.2 x 86 mm -> 308 x 87 mm
- board text removed: "JLCJLCJLCJLC"

Commit message: component placement
Parts:
- removed I2C1, I2C2: Conn_01x04_Female, zzkeeb:Pointing_Cirque-adapter
- added H13: MountingHole, zzkeeb:Hole_M2-spacer, F.Cu at (186.0, 129.0)
- added H14: MountingHole, zzkeeb:Hole_M2-spacer, F.Cu at (252.0, 75.0)
- added H15: MountingHole, zzkeeb:Hole_M2-spacer, F.Cu at (301.0, 97.5)
- added H16: MountingHole, zzkeeb:Hole_M2-spacer, F.Cu at (219.5, 95.0)
- added REF**: Display_1.69inch, zzkeeb:Display_1.69inch, F.Cu at (207.0, 96.5)
- added REF**: Display_1.69inch, zzkeeb:Display_1.69inch, F.Cu at (151.0, 96.5)
- DISP1, DISP2: value Conn_01x08_Female -> Display_generic-spi-8pin; footprint zzkeeb:Connector_JST_PH_S8B-PH-K_1x08_P2.00mm_Horizontal -> zzkeeb:Connector_Display-8pin-SPI-2.0mm
- ROLL1, ROLL2: value roller -> RollerEncoder_EVQWGD001
- TRRS1, TRRS2: value MJ-4PP-9 -> AudioJack4
- USB1, USB2: value USB_C_Receptacle_USB2.0 -> Connector_HRO-TYPE-C-31-M-12; footprint zzkeeb:Connector_USB-C-mid-mount-ali-data -> zzkeeb:Connector_HRO-TYPE-C-31-M-12-data
- moved H7 222.0 mm to (94.0, 126.0)
- moved H10 132.4 mm to (317.0, 132.5)
- moved H8 105.0 mm to (138.5, 95.0)
- moved H1 48.3 mm to (172.0, 129.0)
- moved H5 37.4 mm to (172.0, 95.0)
- moved H11 35.9 mm to (186.0, 95.0)
- moved H2 27.6 mm to (41.0, 132.5)
- moved CIRQUE2 24.4 mm to (142.0, 119.5), turned to 180 degrees
- moved CIRQUE4 23.8 mm to (216.0, 106.0), turned to 0 degrees
- moved DISP2 18.3 mm to (214.0, 130.0), turned to 180 degrees
- moved D31 17.6 mm to (308.2, 126.8), turned to -10 degrees
- moved D36 16.6 mm to (326.4, 126.8), turned to -10 degrees
- moved CIRQUE1 16.5 mm to (158.0, 113.5)
- moved USB2 16.2 mm to (181.0, 113.0)
- moved D39 15.4 mm to (236.4, 142.4), turned to 10 degrees
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Connections:
- net MISO/DC renamed MISO
- net MISO/DC_r renamed MISO_r
- DISP1 pad 1: VCC -> GND
- DISP1 pad 2: GND -> VCC
- DISP1 pad 3: MOSI/SCL -> SCLK/SDA
- DISP1 pad 4: SCLK/SDA -> MOSI/SCL
- DISP1 pad 5: CS -> RST
- DISP1 pad 7: RST -> CS
- DISP2 pad 1: VDD -> GNDA
- DISP2 pad 2: GNDA -> VDD
- DISP2 pad 3: MOSI/SCL_r -> SCLK/SDA_r
- DISP2 pad 4: SCLK/SDA_r -> MOSI/SCL_r
- DISP2 pad 5: CS_r -> RST_r
- DISP2 pad 7: RST_r -> CS_r
- MCU1 pad 15: row3 -> BL
- MCU1 pad 16: row2 -> row3
- MCU1 pad 17: row1 -> row2
- MCU1 pad 18: row0 -> row1
- MCU1 pad 19: BL -> row0
- MCU2 pad 15: row3_r -> BL_r
- MCU2 pad 16: row2_r -> row3_r
- MCU2 pad 17: row1_r -> row2_r
- MCU2 pad 18: row0_r -> row1_r
- MCU2 pad 19: BL_r -> row0_r
Other:
- board size 308 x 87 mm -> 321 x 83.7 mm

Commit message: pcb left side
Parts:
- moved D37 12.5 mm to (272.8, 136.4), turned to 0 degrees
- moved D17 8.50 mm to (85.5, 136.0)
- moved REF** 0.70 mm to (151.6, 96.9)
- moved REF** 0.70 mm to (207.6, 96.9)
- moved LED9 0.14 mm to (50.4, 119.0)
- moved SW11 0.12 mm to (51.2, 123.7)
- moved SW1 0.10 mm to (30.0, 107.1)
- moved LED8 0.08 mm to (32.1, 119.2)
- moved LED7 0.08 mm to (29.2, 102.5)
- moved SW16 0.08 mm to (32.9, 123.8)
- moved SW6 0.07 mm to (48.2, 106.9)
Routing:
- net VCC: track 0.00 -> 534.8 mm, vias 0 -> 21
- net col0: track 0.00 -> 241.2 mm, vias 0 -> 4
- net col1: track 0.00 -> 200.8 mm, vias 0 -> 3
- net col2: track 0.00 -> 187.3 mm, vias 0 -> 5
- net row3: track 0.00 -> 184.6 mm, vias 0 -> 1
- net col3: track 0.00 -> 182.5 mm, vias 0 -> 5
- net col4: track 0.00 -> 161.0 mm, vias 0 -> 5
- net row0: track 0.00 -> 148.5 mm, vias 0 -> 2
- net ENCA: track 0.00 -> 143.1 mm, vias 0 -> 1
- net ENCB: track 0.00 -> 135.7 mm, vias 0 -> 1
- net row2: track 0.00 -> 134.3 mm
- net row1: track 0.00 -> 118.1 mm
- net CS: track 0.00 -> 102.6 mm, vias 0 -> 1
- net SCLK/SDA: track 0.00 -> 86.1 mm, vias 0 -> 1
- net MISO: track 0.00 -> 85.9 mm, vias 0 -> 1
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- added copper zone on B.Cu, net GND
- added copper zone on F.Cu, net GND
Other:
- board size 321 x 83.7 mm -> 321 x 84.6 mm
