File: pcb/choc/pcb.kicad_sch (KiCad schematic)
At the start: 71 parts, among them J1 MJ-4PP-9, J2 USB_C_Receptacle_USB2.0, J3 Conn_01x04_Female, J4 Conn_01x08_Female, J5 Conn_01x12_Female, SW1 SW_PUSH, SW10 SW_PUSH, SW11 SW_PUSH, SW12 SW_PUSH, SW13 SW_PUSH, SW14 SW_PUSH, SW15 SW_PUSH, SW16 SW_PUSH, SW17 SW_PUSH, SW18 SW_PUSH, SW19 SW_PUSH, SW2 SW_PUSH, SW3 SW_PUSH, SW4 SW_PUSH, SW5 SW_PUSH, SW6 SW_PUSH, SW7 SW_PUSH, SW8 SW_PUSH, SW9 SW_PUSH, U1 rp2040-zero, U2 rp2040-zero, U3 roller

Commit message: non-reversible schematic
Parts:
- added D21, D22, D23, D24, D25, D26, D27, D28, D29, D30, D31, D32, D33, D34, D35, D36, D37, D38, D39, D40: D_Small, zzkeeb:Diode_1N4148-SOD123, symbol Device:D_Small
- added H1, H11, H12, H2, H3, H4, H5, H6: MountingHole, zzkeeb:Hole_M2-spacer, symbol Mechanical:MountingHole
- added J10: Conn_01x08_Female, Connector_JST:JST_PH_S8B-PH-K_1x08_P2.00mm_Horizontal, symbol Connector:Conn_01x08_Female
- added J6: MJ-4PP-9, zzkeeb:Connector_TRRS, symbol kbd:MJ-4PP-9
- added J7: USB_C_Receptacle_USB2.0, zzkeeb:Connector_USB-C-mid-mount-ali-data, symbol Connector:USB_C_Receptacle_USB2.0
- added J8: Conn_01x12_Female, symbol Connector:Conn_01x12_Female
- added J9: Conn_01x04_Female, zzkeeb:Pointing_Cirque-adapter, symbol Connector:Conn_01x04_Female
- added LED1, LED10, LED11, LED12, LED13, LED14, LED15, LED16, LED17, LED18, LED19, LED2, LED3, LED4, LED5, LED6, LED7, LED8, LED9: YS-SK6812MINI-E, zzkeeb:LED_SK6812-MINI-E, symbol kbd:YS-SK6812MINI-E
- added RE1: RotaryEncoder_Switch, zzkeeb:RotaryEncoder_EC11, symbol Device:RotaryEncoder_Switch
- added SW20, SW21, SW22, SW23, SW24, SW25, SW26, SW27, SW28, SW29, SW30, SW31, SW32, SW33, SW34, SW35, SW36, SW37, SW38: SW_PUSH, zzkeeb:Switch_ChocV1-hotswap, symbol kbd:SW_PUSH
- added U3: roller, zzkeeb:RotaryEncoder_EVQWGD001, symbol zzkeeb:RollerEncoder_EVQWGD001
- D1, D10, D11, D12, D13, D14, D15, D16, D17, D18, D19, D2, D20, D3, D4, D5, D6, D7, D8, D9: footprint zzkeeb:Diode_1N4148-SOD123-reversible -> zzkeeb:Diode_1N4148-SOD123
- J1: footprint zzkeeb:Connector_TRRS-reversible -> zzkeeb:Connector_TRRS
- J2: footprint zzkeeb:Connector_USB-C-mid-mount-ali-reversible-data -> zzkeeb:Connector_USB-C-mid-mount-ali-data
- LED20: renamed from LED1; footprint zzkeeb:LED_SK6812-MINI-E-reversible -> zzkeeb:LED_SK6812-MINI-E
- LED21: renamed from LED2; footprint zzkeeb:LED_SK6812-MINI-E-reversible -> zzkeeb:LED_SK6812-MINI-E
- LED22: renamed from LED3; footprint zzkeeb:LED_SK6812-MINI-E-reversible -> zzkeeb:LED_SK6812-MINI-E
- LED23: renamed from LED4; footprint zzkeeb:LED_SK6812-MINI-E-reversible -> zzkeeb:LED_SK6812-MINI-E
- LED24: renamed from LED5; footprint zzkeeb:LED_SK6812-MINI-E-reversible -> zzkeeb:LED_SK6812-MINI-E
- LED25: renamed from LED6; footprint zzkeeb:LED_SK6812-MINI-E-reversible -> zzkeeb:LED_SK6812-MINI-E
- LED26: renamed from LED7; footprint zzkeeb:LED_SK6812-MINI-E-reversible -> zzkeeb:LED_SK6812-MINI-E
- LED27: renamed from LED8; footprint zzkeeb:LED_SK6812-MINI-E-reversible -> zzkeeb:LED_SK6812-MINI-E
- LED28: renamed from LED9; footprint zzkeeb:LED_SK6812-MINI-E-reversible -> zzkeeb:LED_SK6812-MINI-E
- LED29: renamed from LED10; footprint zzkeeb:LED_SK6812-MINI-E-reversible -> zzkeeb:LED_SK6812-MINI-E
- LED30: renamed from LED11; footprint zzkeeb:LED_SK6812-MINI-E-reversible -> zzkeeb:LED_SK6812-MINI-E
- LED31: renamed from LED12; footprint zzkeeb:LED_SK6812-MINI-E-reversible -> zzkeeb:LED_SK6812-MINI-E
- LED32: renamed from LED13; footprint zzkeeb:LED_SK6812-MINI-E-reversible -> zzkeeb:LED_SK6812-MINI-E
- LED33: renamed from LED14; footprint zzkeeb:LED_SK6812-MINI-E-reversible -> zzkeeb:LED_SK6812-MINI-E
- LED34: renamed from LED15; footprint zzkeeb:LED_SK6812-MINI-E-reversible -> zzkeeb:LED_SK6812-MINI-E
- LED35: renamed from LED16; footprint zzkeeb:LED_SK6812-MINI-E-reversible -> zzkeeb:LED_SK6812-MINI-E
- LED36: renamed from LED17; footprint zzkeeb:LED_SK6812-MINI-E-reversible -> zzkeeb:LED_SK6812-MINI-E
- LED37: renamed from LED18; footprint zzkeeb:LED_SK6812-MINI-E-reversible -> zzkeeb:LED_SK6812-MINI-E
- LED38: renamed from LED19; footprint zzkeeb:LED_SK6812-MINI-E-reversible -> zzkeeb:LED_SK6812-MINI-E
- SW1, SW10, SW11, SW12, SW13, SW14, SW15, SW16, SW17, SW18, SW19, SW2, SW3, SW4, SW5, SW6, SW7, SW8, SW9: footprint zzkeeb:Switch_ChocV1-hotswap-reversible -> zzkeeb:Switch_ChocV1-hotswap
- U1, U2: footprint zzkeeb:MCU_rp2040-zero-smd -> zzkeeb:MCU_rp2040-zero-tht-pads
- renumbered H4 to H10, H1 to H7, H2 to H8, H3 to H9, J5 to J3, J3 to J4, J4 to J5, RE1 to RE2, U3 to U4
Connections:
- net BL: now also U1.19 (28); no longer U1.8 (7), U2.8 (7)
- net CS: no longer U2.6 (5)
- net ENCA: now also U1.8 (7), RE1.A, U3.A; no longer RE2.A, U1.15 (14), U2.9 (8), U4.A
- net ENCB: now also RE1.B, U3.B; no longer RE2.B, U2.15 (14), U4.B
- net GND: now also LED1.3 (VSS), LED10.3 (VSS), LED11.3 (VSS), LED12.3 (VSS), LED13.3 (VSS), LED14.3 (VSS), LED15.3 (VSS), LED16.3 (VSS), LED17.3 (VSS), LED18.3 (VSS), LED19.3 (VSS), LED2.3 (VSS), LED3.3 (VSS), LED4.3 (VSS), LED5.3 (VSS), LED6.3 (VSS), LED7.3 (VSS), LED8.3 (VSS), LED9.3 (VSS), RE1.C, U3.C; no longer LED20.3 (VSS), LED21.3 (VSS), LED22.3 (VSS), LED23.3 (VSS), LED24.3 (VSS), LED25.3 (VSS), LED26.3 (VSS), LED27.3 (VSS), LED28.3 (VSS), LED29.3 (VSS), LED30.3 (VSS), LED31.3 (VSS), LED32.3 (VSS), LED33.3 (VSS), LED34.3 (VSS), LED35.3 (VSS), LED36.3 (VSS), LED37.3 (VSS), LED38.3 (VSS), RE2.C, U2.22 (GND), U4.C
- net LED: now also U1.20 (29), LED1.4 (DIN); no longer LED20.4 (DIN), U1.16 (15), U2.16 (15)
- net MISO/DC: no longer U2.5 (4)
- net MOSI/SCL: no longer U2.4 (3)
- net RST: no longer U2.7 (6)
- net RX: no longer U2.2 (1)
- net SCLK/SDA: no longer U2.3 (2)
- net SW_ENCA: now also RE1.S2, U3.S2; no longer RE2.S2, U4.S2
- net TX: no longer U2.1 (0)
- net VCC: now also LED1.1 (VDD), LED10.1 (VDD), LED11.1 (VDD), LED12.1 (VDD), LED13.1 (VDD), LED14.1 (VDD), LED15.1 (VDD), LED16.1 (VDD), LED17.1 (VDD), LED18.1 (VDD), LED19.1 (VDD), LED2.1 (VDD), LED3.1 (VDD), LED4.1 (VDD), LED5.1 (VDD), LED6.1 (VDD), LED7.1 (VDD), LED8.1 (VDD), LED9.1 (VDD); no longer LED20.1 (VDD), LED21.1 (VDD), LED22.1 (VDD), LED23.1 (VDD), LED24.1 (VDD), LED25.1 (VDD), LED26.1 (VDD), LED27.1 (VDD), LED28.1 (VDD), LED29.1 (VDD), LED30.1 (VDD), LED31.1 (VDD), LED32.1 (VDD), LED33.1 (VDD), LED34.1 (VDD), LED35.1 (VDD), LED36.1 (VDD), LED37.1 (VDD), LED38.1 (VDD), U2.21 (3V3)
- net col0: no longer U2.14 (13)
- net col1: now also RE1.S1, U3.S1; no longer RE2.S1, U2.13 (12), U4.S1
- net col2: no longer U2.12 (11)
- net col3: no longer U2.11 (10)
- net col4: no longer U2.10 (9)
- net row0: now also U1.15 (14); no longer U1.17 (26), U2.17 (26)
- net row1: now also U1.16 (15); no longer U1.18 (27), U2.18 (27)
- net row2: now also U1.17 (26); no longer U1.19 (28), U2.19 (28)
- net row3: now also U1.18 (27); no longer U1.20 (29), U2.20 (29)
- new net: D28.2 (A), SW27.1
- new net: D26.2 (A), SW25.1
- new net: D33.2 (A), SW32.1
- new net: D24.2 (A), SW23.1
- new net: D30.2 (A), SW29.1
- new net: LED15.2 (DOUT), LED16.4 (DIN)
- new net: LED14.2 (DOUT), LED15.4 (DIN)
- new net: D25.2 (A), SW24.1
- new net: D29.2 (A), SW28.1
- new net: D21.2 (A), SW20.1
- new net: D38.2 (A), SW36.1
- new net: D36.2 (A), SW35.1
- new net: LED2.2 (DOUT), LED3.4 (DIN)
- new net: LED1.2 (DOUT), LED2.4 (DIN)
- new net: D27.2 (A), SW26.1
- new net: LED18.2 (DOUT), LED19.4 (DIN)
- new net: D32.2 (A), SW31.1
- new net: D39.2 (A), SW37.1
- new net: D40.2 (A), SW38.1
- new net: LED12.2 (DOUT), LED13.4 (DIN)
- new net: LED11.2 (DOUT), LED12.4 (DIN)
- new net: LED13.2 (DOUT), LED14.4 (DIN)
- new net: D31.2 (A), SW30.1
- new net: D22.2 (A), SW21.1
- new net: D35.2 (A), SW34.1
- new net: LED5.2 (DOUT), LED6.4 (DIN)
- new net: LED4.2 (DOUT), LED5.4 (DIN)
- new net: D23.2 (A), SW22.1
- new net: LED8.2 (DOUT), LED9.4 (DIN)
- new net: LED7.2 (DOUT), LED8.4 (DIN)
- new net: LED10.4 (DIN), LED9.2 (DOUT)
- new net: LED10.2 (DOUT), LED11.4 (DIN)
- new net: LED3.2 (DOUT), LED4.4 (DIN)
- new net: LED17.2 (DOUT), LED18.4 (DIN)
- new net: LED16.2 (DOUT), LED17.4 (DIN)
- new net: D34.2 (A), SW33.1
- new net: LED6.2 (DOUT), LED7.4 (DIN)
- new net BL_r: J10.8 (Pin_8), U2.19 (28)
- new net CS_r: J10.5 (Pin_5), J8.11 (Pin_11), U2.6 (5)
- new net ENCA_r: RE2.A, U2.8 (7), U4.A
- new net ENCB_r: RE2.B, U2.9 (8), U4.B
- new net GNDA: J10.2 (Pin_2), J6.C, J7.A1 (GND), J7.A12 (GND), J7.B1 (GND), J7.B12 (GND), J8.2 (Pin_2), J9.4 (Pin_4), LED20.3 (VSS), LED21.3 (VSS), LED22.3 (VSS), LED23.3 (VSS), LED24.3 (VSS), LED25.3 (VSS), LED26.3 (VSS), LED27.3 (VSS), LED28.3 (VSS), LED29.3 (VSS), LED30.3 (VSS), LED31.3 (VSS), LED32.3 (VSS), LED33.3 (VSS), LED34.3 (VSS), LED35.3 (VSS), LED36.3 (VSS), LED37.3 (VSS), LED38.3 (VSS), RE2.C, U2.22 (GND), U4.C
- new net LED_r: LED20.4 (DIN), U2.20 (29)
- new net MISO/DC_r: J10.6 (Pin_6), J8.10 (Pin_10), U2.5 (4)
- new net MOSI/SCL_r: J10.3 (Pin_3), J8.4 (Pin_4), J8.8 (Pin_8), J9.2 (Pin_2), U2.4 (3)
- new net RST_r: J10.7 (Pin_7), U2.7 (6)
- new net RX_r: J6.B, J7.A6 (D+), J7.B6 (D+), U2.2 (1)
- new net SCLK/SDA_r: J10.4 (Pin_4), J8.12 (Pin_12), J8.3 (Pin_3), J9.1 (Pin_1), U2.3 (2)
- new net SW_ENCA_r: D37.2 (A), RE2.S2, U4.S2
- new net TX_r: J6.A, J7.A7 (D-), J7.B7 (D-), U2.1 (0)
- new net VDD: J10.1 (Pin_1), J6.D, J7.A4 (VBUS), J7.A9 (VBUS), J7.B4 (VBUS), J7.B9 (VBUS), J8.1 (Pin_1), J9.3 (Pin_3), LED20.1 (VDD), LED21.1 (VDD), LED22.1 (VDD), LED23.1 (VDD), LED24.1 (VDD), LED25.1 (VDD), LED26.1 (VDD), LED27.1 (VDD), LED28.1 (VDD), LED29.1 (VDD), LED30.1 (VDD), LED31.1 (VDD), LED32.1 (VDD), LED33.1 (VDD), LED34.1 (VDD), LED35.1 (VDD), LED36.1 (VDD), LED37.1 (VDD), LED38.1 (VDD), U2.21 (3V3)
- new net col0_r: SW20.2, SW25.2, SW30.2, SW35.2, U2.10 (9)
- new net col1_r: RE2.S1, SW21.2, SW26.2, SW31.2, U2.11 (10), U4.S1
- new net col2_r: SW22.2, SW27.2, SW32.2, SW36.2, U2.12 (11)
- new net col3_r: SW23.2, SW28.2, SW33.2, SW37.2, U2.13 (12)
- new net col4_r: SW24.2, SW29.2, SW34.2, SW38.2, U2.14 (13)
- new net row0_r: D21.1 (K), D22.1 (K), D23.1 (K), D24.1 (K), D25.1 (K), U2.15 (14)
- new net row1_r: D26.1 (K), D27.1 (K), D28.1 (K), D29.1 (K), D30.1 (K), U2.16 (15)
- new net row2_r: D31.1 (K), D32.1 (K), D33.1 (K), D34.1 (K), D35.1 (K), U2.17 (26)
- new net row3_r: D36.1 (K), D37.1 (K), D38.1 (K), D39.1 (K), D40.1 (K), U2.18 (27)
- no-connect marks 13 -> 24
Other:
- moved on the sheet: D1, D10, D11, D12, D13, D14, D15, D16, D17, D18, D19, D2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

Commit message: prototype 0
Parts:
- removed D20, D21, D22, D23, D24, D25, D26, D27, D28, D29, D30, D31, D32, D33, D34, D35, D36, D37, D38, D39, D40: D_Small, zzkeeb:Diode_1N4148-SOD123, symbol Device:D_Small
- removed H10, H11, H12, H5, H6, H7, H8, H9: MountingHole, zzkeeb:Hole_M2-spacer, symbol Mechanical:MountingHole
- removed J1, J6: MJ-4PP-9, zzkeeb:Connector_TRRS, symbol kbd:MJ-4PP-9
- removed J10, J5: Conn_01x08_Female, Connector_JST:JST_PH_S8B-PH-K_1x08_P2.00mm_Horizontal, symbol Connector:Conn_01x08_Female
- removed J3, J8: Conn_01x12_Female, symbol Connector:Conn_01x12_Female
- removed J4, J9: Conn_01x04_Female, zzkeeb:Pointing_Cirque-adapter, symbol Connector:Conn_01x04_Female
- removed J7: USB_C_Receptacle_USB2.0, zzkeeb:Connector_USB-C-mid-mount-ali-data, symbol Connector:USB_C_Receptacle_USB2.0
- removed LED1, LED10, LED11, LED12, LED13, LED14, LED15, LED16, LED17, LED18, LED19, LED2, LED20, LED21, LED22, LED23, LED24, LED25, LED26, LED27, LED28, LED29, LED3, LED30, LED31, LED32, LED33, LED34, LED35, LED36, LED37, LED38, LED4, LED5, LED6, LED7, LED8, LED9: YS-SK6812MINI-E, zzkeeb:LED_SK6812-MINI-E, symbol kbd:YS-SK6812MINI-E
- removed RE2: RotaryEncoder_Switch, zzkeeb:RotaryEncoder_EC11, symbol Device:RotaryEncoder_Switch
- removed SW1, SW10, SW11, SW12, SW13, SW14, SW15, SW16, SW17, SW18, SW19, SW2, SW20, SW21, SW22, SW23, SW24, SW25, SW26, SW27, SW28, SW29, SW3, SW30, SW31, SW32, SW33, SW34, SW35, SW36, SW37, SW38, SW4, SW5, SW6, SW7, SW8, SW9: SW_PUSH, zzkeeb:Switch_ChocV1-hotswap, symbol kbd:SW_PUSH
- removed U1, U2: rp2040-zero, zzkeeb:MCU_rp2040-zero-tht-pads, symbol kleeb-mcu:rp2040-zero
- removed U4: roller, zzkeeb:RotaryEncoder_EVQWGD001, symbol zzkeeb:RollerEncoder_EVQWGD001
- added J1: AudioJack4, zzkeeb:Connector_TRRS-reversible, symbol Connector:AudioJack4
- added LED1, LED10, LED11, LED12, LED13, LED14, LED15, LED16, LED17, LED18, LED2, LED3, LED4, LED5, LED6, LED7, LED8, LED9: LED_SK6812MINI-E, zzkeeb:LED_SK6812-MINI-E-reversible, symbol zzkeeb:LED_SK6812MINI-E
- added SW1, SW10, SW11, SW12, SW13, SW14, SW15, SW16, SW17, SW18, SW2, SW3, SW4, SW5, SW6, SW7, SW8, SW9: Switch, zzkeeb:Switch_ChocV1-hotswap-reversible, symbol zzkeeb:Switch
- added U1, U2: MCU_rp2040-zero, zzkeeb:MCU_rp2040-zero-smd, symbol zzkeeb:MCU_rp2040-zero
- D1, D10, D11, D12, D13, D14, D15, D16, D17, D18, D19, D2, D3, D4, D5, D6, D7, D8, D9: footprint zzkeeb:Diode_1N4148-SOD123 -> zzkeeb:Diode_1N4148-SOD123-reversible
- J2: footprint zzkeeb:Connector_USB-C-mid-mount-ali-data -> zzkeeb:Connector_USB-C-mid-mount-ali-reversible-data
- U3: value roller -> RollerEncoder_EVQWGD001
Connections:
- net ENCA: now also U1.17 (26), U2.7 (6)
- net ENCB: now also U1.7 (6), U2.17 (26)
- net GND: now also J1.R1, LED1.3 (VSS), LED10.3 (VSS), LED11.3 (VSS), LED12.3 (VSS), LED13.3 (VSS), LED14.3 (VSS), LED15.3 (VSS), LED16.3 (VSS), LED17.3 (VSS), LED18.3 (VSS), LED2.3 (VSS), LED3.3 (VSS), LED4.3 (VSS), LED5.3 (VSS), LED6.3 (VSS), LED7.3 (VSS), LED8.3 (VSS), LED9.3 (VSS), U1.22 (GND), U2.22 (GND)
- net LED: now also LED1.4 (DIN), U1.19 (28), U2.19 (28)
- net RX: now also J1.R2, U1.2 (1), U2.2 (1)
- net SW_ENCA: now also D16.2 (A); no longer D17.2 (A)
- net TX: now also J1.S, U1.1 (0), U2.1 (0)
- net VCC: now also J1.T, LED1.1 (VDD), LED10.1 (VDD), LED11.1 (VDD), LED12.1 (VDD), LED13.1 (VDD), LED14.1 (VDD), LED15.1 (VDD), LED16.1 (VDD), LED17.1 (VDD), LED18.1 (VDD), LED2.1 (VDD), LED3.1 (VDD), LED4.1 (VDD), LED5.1 (VDD), LED6.1 (VDD), LED7.1 (VDD), LED8.1 (VDD), LED9.1 (VDD), U1.21 (3V3), U2.21 (3V3)
- net col0: now also SW10.2, SW15.2, SW5.2, U1.10 (9), U2.14 (13)
- net col1: now also SW1.2, SW11.2, SW6.2, U1.11 (10), U2.13 (12)
- net col2: now also SW12.2, SW16.2, SW2.2, SW7.2, U1.12 (11), U2.12 (11)
- net col3: now also SW13.2, SW17.2, SW3.2, SW8.2, U1.13 (12), U2.11 (10)
- net col4: now also SW14.2, SW18.2, SW4.2, SW9.2, U1.14 (13), U2.10 (9)
- net row0: now also U1.16 (15), U2.8 (7); no longer D5.1 (K)
- net row1: now also D5.1 (K), U1.15 (14), U2.9 (8); no longer D10.1 (K)
- net row2: now also D10.1 (K), U1.9 (8), U2.15 (14); no longer D15.1 (K)
- net row3: now also D15.1 (K), U1.8 (7), U2.16 (15)
- net at D10.2 (A): now also SW10.1
- net at D11.2 (A): now also SW11.1
- net at D12.2 (A): now also SW12.1
- net at D9.2 (A): now also SW9.1
- net at D19.2 (A): now also SW18.1
- net at D8.2 (A): now also SW8.1
- net at D7.2 (A): now also SW7.1
- net at D14.2 (A): now also SW14.1
- net at D2.2 (A): now also SW2.1
- net at D6.2 (A): now also SW6.1
- net at D15.2 (A): now also SW15.1
- net at D13.2 (A): now also SW13.1
- net at D3.2 (A): now also SW3.1
- net at D5.2 (A): now also SW5.1
- net at D4.2 (A): now also SW4.1
- net at D18.2 (A): now also SW17.1
- net at D1.2 (A): now also SW1.1
- new net: LED2.2 (DOUT), LED3.4 (DIN)
- new net: LED1.2 (DOUT), LED2.4 (DIN)
- new net: LED10.2 (DOUT), LED11.4 (DIN)
- new net: LED10.4 (DIN), LED5.2 (DOUT)
- new net: LED12.2 (DOUT), LED13.4 (DIN)
- new net: LED11.2 (DOUT), LED12.4 (DIN)
- new net: D17.2 (A), SW16.1
- new net: LED8.4 (DIN), LED9.2 (DOUT)
- new net: LED4.2 (DOUT), LED9.4 (DIN)
- new net: LED17.4 (DIN), LED18.2 (DOUT)
- new net: LED14.2 (DOUT), LED18.4 (DIN)
- new net: LED13.2 (DOUT), LED14.4 (DIN)
- new net: LED3.2 (DOUT), LED4.4 (DIN)
- new net: LED16.4 (DIN), LED17.2 (DOUT)
- new net: LED5.4 (DIN), LED6.2 (DOUT)
- new net: LED7.4 (DIN), LED8.2 (DOUT)
- new net: LED15.4 (DIN), LED16.2 (DOUT)
- new net: LED6.4 (DIN), LED7.2 (DOUT)
- no-connect marks 24 -> 21

Commit message: small fix
Parts:
- D1, D10, D11, D12, D13, D14, D15, D16, D17, D18, D19, D2, D3, D4, D5, D6, D7, D8, D9: footprint zzkeeb:Diode_1N4148-SOD123-reversible -> zzkeeb:Diode_1N4148-SOD123-reversible-flip3d
- RE1: footprint zzkeeb:RotaryEncoder_EC11 -> zzkeeb:RotaryEncoder_EC11-reversible
