File: pcb/choc/pcb.kicad_sch (KiCad schematic)
At the start: 152 parts, among them SW1 Switch, SW10 Switch, SW11 Switch, SW12 Switch, SW13 Switch, SW14 Switch, SW15 Switch, SW16 Switch, SW17 Switch, SW18 Switch, SW19 Switch, SW2 Switch, SW20 Switch, SW21 Switch, SW22 Switch, SW23 Switch, SW24 Switch, SW25 Switch, SW26 Switch, SW27 Switch, SW28 Switch, SW29 Switch, SW3 Switch, SW30 Switch, SW31 Switch, SW32 Switch, SW33 Switch, SW34 Switch, SW35 Switch, SW36 Switch, SW37 Switch, SW38 Switch, SW4 Switch, SW5 Switch, SW6 Switch, SW7 Switch, SW8 Switch, SW9 Switch

Commit message: add pull up resistors, additional holes
Parts:
- added H17, H18, H19, H20: MountingHole, zzkeeb:Hole_M2-spacer, symbol Mechanical:MountingHole
- added R1, R2, R3, R4: R, Resistor_SMD:R_1206_3216Metric_Pad1.30x1.75mm_HandSolder, symbol Device:R
Connections:
- net MOSI/SCL: now also R1.2
- net MOSI/SCL_r: now also R3.2
- net SCLK/SDA: now also R2.2
- net SCLK/SDA_r: now also R4.2
- net VCC: now also R1.1, R2.1
- net VDD: now also R3.1, R4.1
Other:
- moved on the sheet: H1, H10, H11, H12, H13, H14, H15, H16, H2, H3, H4, H5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

Commit message: another resize
Parts:
- removed H11, H16, H18, H20, H5, H8: MountingHole, zzkeeb:Hole_M2-spacer, symbol Mechanical:MountingHole
Changed lines of the file:
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@@
     )
   )
-  (symbol (lib_id "Mechanical:MountingHole") (at 132.08 240.03 0) (unit 1)
-    (in_bom yes) (on_board yes) (dnp no) (fields_autoplaced)
-    (property "Reference" "H5" (at 134.62 238.7599 0)
-      (effects (font (size 1.27 1.27)) (justify left))
-    )
-    (property "Value" "MountingHole" (at 134.62 241.2999 0)
-      (effects (font (size 1.27 1.27)) (justify left))
-    )
-    (property "Footprint" "zzkeeb:Hole_M2-spacer" (at 132.08 240.03 0)
-      (effects (font (size 1.27 1.27)) hide)
-    )
-    (property "Datasheet" "~" (at 132.08 240.03 0)
-      (effects (font (size 1.27 1.27)) hide)
-    )
-    (instances
-      (project "pcb"
-        (path "/5689f24b-6eca-4ca4-9c6c-dd56b6ced5a9"
-          (reference "H5") (unit 1)
-        )
-      )
-    )
-  )
   (symbol (lib_id "power:VDD") (at 269.24 44.45 0) (unit 1)
     (in_bom yes) (on_board yes) (dnp no)
@@
     )
   )
-  (symbol (lib_id "Mechanical:MountingHole") (at 339.09 243.84 0) (unit 1)
-    (in_bom yes) (on_board yes) (dnp no) (fields_autoplaced)
-    (property "Reference" "H20" (at 341.63 242.5699 0)
-      (effects (font (size 1.27 1.27)) (justify left))
-    )
-    (property "Value" "MountingHole" (at 341.63 245.1099 0)
-      (effects (font (size 1.27 1.27)) (justify left))
-    )
-    (property "Footprint" "zzkeeb:Hole_M2-spacer" (at 339.09 243.84 0)
-      (effects (font (size 1.27 1.27)) hide)
-    )
-    (property "Datasheet" "~" (at 339.09 243.84 0)
-      (effects (font (size 1.27 1.27)) hide)
-    )
-    (instances
-      (project "pcb"
-        (path "/5689f24b-6eca-4ca4-9c6c-dd56b6ced5a9"
-          (reference "H20") (unit 1)
-        )
-      )
-    )
-  )
   (symbol (lib_id "zzkeeb:Switch") (at 307.34 113.03 0) (unit 1)
     (in_bom yes) (on_board yes) (dnp no) (fields_autoplaced)
@@
     )
   )
-  (symbol (lib_id "Mechanical:MountingHole") (at 339.09 199.39 0) (unit 1)
-    (in_bom yes) (on_board yes) (dnp no) (fields_autoplaced)
-    (property "Reference" "H11" (at 341.63 198.1199 0)
-      (effects (font (size 1.27 1.27)) (justify left))
-    )
-    (property "Value" "MountingHole" (at 341.63 200.6599 0)
-      (effects (font (size 1.27 1.27)) (justify left))
-    )
-    (property "Footprint" "zzkeeb:Hole_M2-spacer" (at 339.09 199.39 0)
-      (effects (font (size 1.27 1.27)) hide)
-    )
-    (property "Datasheet" "~" (at 339.09 199.39 0)
-      (effects (font (size 1.27 1.27)) hide)
-    )
-    (instances
-      (project "pcb"
-        (path "/5689f24b-6eca-4ca4-9c6c-dd56b6ced5a9"
-          (reference "H11") (unit 1)
-        )
-      )
-    )
-  )
   (symbol (lib_id "zzkeeb:LED_SK6812MINI-E") (at 100.33 232.41 0) (unit 1)
     (in_bom yes) (on_board yes) (dnp no)
@@
     )
   )
-  (symbol (lib_id "Mechanical:MountingHole") (at 339.09 231.14 0) (unit 1)
-    (in_bom yes) (on_board yes) (dnp no) (fields_autoplaced)
-    (property "Reference" "H16" (at 341.63 229.8699 0)
-      (effects (font (size 1.27 1.27)) (justify left))
-    )
-    (property "Value" "MountingHole" (at 341.63 232.4099 0)
-      (effects (font (size 1.27 1.27)) (justify left))
-    )
-    (property "Footprint" "zzkeeb:Hole_M2-spacer" (at 339.09 231.14 0)
-      (effects (font (size 1.27 1.27)) hide)
-    )
-    (property "Datasheet" "~" (at 339.09 231.14 0)
-      (effects (font (size 1.27 1.27)) hide)
-    )
-    (instances
-      (project "pcb"
-        (path "/5689f24b-6eca-4ca4-9c6c-dd56b6ced5a9"
-          (reference "H16") (unit 1)
-        )
-      )
-    )
-  )
   (symbol (lib_id "zzkeeb:Switch") (at 271.78 153.67 0) (unit 1)
     (in_bom yes) (on_board yes) (dnp no) (fields_autoplaced)
@@
     )
   )
-  (symbol (lib_id "Mechanical:MountingHole") (at 132.08 271.78 0) (unit 1)
-    (in_bom yes) (on_board yes) (dnp no) (fields_autoplaced)
-    (property "Reference" "H18" (at 134.62 270.5099 0)
-      (effects (font (size 1.27 1.27)) (justify left))
-    )
-    (property "Value" "MountingHole" (at 134.62 273.0499 0)
-      (effects (font (size 1.27 1.27)) (justify left))
-    )
-    (property "Footprint" "zzkeeb:Hole_M2-spacer" (at 132.08 271.78 0)
-      (effects (font (size 1.27 1.27)) hide)
-    )
-    (property "Datasheet" "~" (at 132.08 271.78 0)
-      (effects (font (size 1.27 1.27)) hide)
-    )
-    (instances
-      (project "pcb"
-        (path "/5689f24b-6eca-4ca4-9c6c-dd56b6ced5a9"
-          (reference "H18") (unit 1)
-        )
-      )
-    )
-  )
   (symbol (lib_id "zzkeeb:Switch") (at 289.56 153.67 0) (unit 1)
     (in_bom yes) (on_board yes) (dnp no) (fields_autoplaced)
@@
         )
       )
-    )
-  )
-  (symbol (lib_id "Mechanical:MountingHole") (at 132.08 259.08 0) (unit 1)
-    (in_bom yes) (on_board yes) (dnp no) (fields_autoplaced)
-    (property "Reference" "H8" (at 134.62 257.8099 0)
-      (effects (font (size 1.27 1.27)) (justify left))
-    )
-    (property "Value" "MountingHole" (at 134.62 260.3499 0)
-      (effects (font (size 1.27 1.27)) (justify left))
-    )
-    (property "Footprint" "zzkeeb:Hole_M2-spacer" (at 132.08 259.08 0)
-      (effects (font (size 1.27 1.27)) hide)
-    )
-    (property "Datasheet" "~" (at 132.08 259.08 0)
-      (effects (font (size 1.27 1.27)) hide)
-    )
-    (instances
-      (project "pcb"
-        (path "/5689f24b-6eca-4ca4-9c6c-dd56b6ced5a9"
-          (reference "H8") (unit 1)
-        )
-      )
