File: pcb/mx40/pcb.kicad_sch (KiCad schematic)
At the start: 172 parts, among them SW1 Switch, SW10 Switch, SW11 Switch, SW12 Switch, SW13 Switch, SW14 Switch, SW15 Switch, SW16 Switch, SW17 Switch, SW18 Switch, SW19 Switch, SW2 Switch, SW20 Switch, SW21 Switch, SW22 Switch, SW23 Switch, SW24 Switch, SW25 Switch, SW26 Switch, SW27 Switch, SW28 Switch, SW29 Switch, SW3 Switch, SW30 Switch, SW31 Switch, SW32 Switch, SW33 Switch, SW34 Switch, SW35 Switch, SW36 Switch, SW37 Switch, SW38 Switch, SW39 Switch, SW4 Switch, SW40 Switch, SW5 Switch, SW6 Switch, SW7 Switch, SW8 Switch, SW9 Switch

Commit message: replace vertical VIK footprint for easier soldering
Parts:
- VIK_K1, VIK_K4: footprint vik:vik-keyboard-connector-vertical -> zzkeeb:Connector_VIK-vertical-keyboard
Changed lines of the file:
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@@
 			)
 		)
-		(property "Footprint" "vik:vik-keyboard-connector-vertical"
+		(property "Footprint" "zzkeeb:Connector_VIK-vertical-keyboard"
 			(at 486.41 250.19 0)
 			(effects
@@
 			)
 		)
-		(property "Footprint" "vik:vik-keyboard-connector-vertical"
+		(property "Footprint" "zzkeeb:Connector_VIK-vertical-keyboard"
 			(at 186.69 251.46 0)
 			(effects
