File: pcb/mx/pcb.kicad_sch (KiCad schematic)
At the start: 166 parts, among them SW1 Switch, SW10 Switch, SW11 Switch, SW12 Switch, SW13 Switch, SW14 Switch, SW15 Switch, SW16 Switch, SW17 Switch, SW18 Switch, SW19 Switch, SW2 Switch, SW20 Switch, SW21 Switch, SW22 Switch, SW23 Switch, SW24 Switch, SW25 Switch, SW26 Switch, SW27 Switch, SW28 Switch, SW29 Switch, SW3 Switch, SW30 Switch, SW31 Switch, SW32 Switch, SW33 Switch, SW34 Switch, SW35 Switch, SW36 Switch, SW37 Switch, SW38 Switch, SW4 Switch, SW5 Switch, SW6 Switch, SW7 Switch, SW8 Switch, SW9 Switch

Commit message: update components
Parts:
- VIK_K1, VIK_K4: footprint zzkeeb:Connector_FFC-FPC-vertical-12pin -> zzkeeb:Connector_VIK-vertical-keyboard
- VIK_K2, VIK_K5: footprint zzkeeb:Connector_FPC-FFC-adapter-12pin -> zzkeeb:Connector_VIK-adapter-keyboard
- VIK_K3, VIK_K6: footprint Connector_FFC-FPC:Hirose_FH12-12S-0.5SH_1x12-1MP_P0.50mm_Horizontal -> zzkeeb:Connector_VIK-horizontal-keyboard
Changed lines of the file:
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@@
       (effects (font (size 1.27 1.27)) (justify left))
     )
-    (property "Footprint" "Connector_FFC-FPC:Hirose_FH12-12S-0.5SH_1x12-1MP_P0.50mm_Horizontal" (at 200.66 347.98 0)
+    (property "Footprint" "zzkeeb:Connector_VIK-horizontal-keyboard" (at 200.66 347.98 0)
       (effects (font (size 1.27 1.27)) hide)
     )
@@
       (effects (font (size 1.27 1.27)) (justify left))
     )
-    (property "Footprint" "zzkeeb:Connector_FPC-FFC-adapter-12pin" (at 238.76 302.26 0)
+    (property "Footprint" "zzkeeb:Connector_VIK-adapter-keyboard" (at 238.76 302.26 0)
       (effects (font (size 1.27 1.27)) hide)
     )
@@
       (effects (font (size 1.27 1.27)) (justify left))
     )
-    (property "Footprint" "Connector_FFC-FPC:Hirose_FH12-12S-0.5SH_1x12-1MP_P0.50mm_Horizontal" (at 497.84 347.98 0)
+    (property "Footprint" "zzkeeb:Connector_VIK-horizontal-keyboard" (at 497.84 347.98 0)
       (effects (font (size 1.27 1.27)) hide)
     )
@@
       (effects (font (size 1.27 1.27)) (justify left))
     )
-    (property "Footprint" "zzkeeb:Connector_FFC-FPC-vertical-12pin" (at 497.84 302.26 0)
+    (property "Footprint" "zzkeeb:Connector_VIK-vertical-keyboard" (at 497.84 302.26 0)
       (effects (font (size 1.27 1.27)) hide)
     )
@@
       (effects (font (size 1.27 1.27)) (justify left))
     )
-    (property "Footprint" "zzkeeb:Connector_FPC-FFC-adapter-12pin" (at 533.4 302.26 0)
+    (property "Footprint" "zzkeeb:Connector_VIK-adapter-keyboard" (at 533.4 302.26 0)
       (effects (font (size 1.27 1.27)) hide)
     )
@@
       (effects (font (size 1.27 1.27)) (justify left))
     )
-    (property "Footprint" "zzkeeb:Connector_FFC-FPC-vertical-12pin" (at 200.66 302.26 0)
+    (property "Footprint" "zzkeeb:Connector_VIK-vertical-keyboard" (at 200.66 302.26 0)
       (effects (font (size 1.27 1.27)) hide)
     )

Commit message: hole updates
Parts:
- H1, H10, H11, H12, H13, H14, H15, H16, H17, H19, H2, H3, H4, H5, H6, H7, H8, H9: footprint zzkeeb:Hole_M2-spacer -> zzkeeb:Hole_M2
Changed lines of the file:
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@@
       (effects (font (size 1.27 1.27)) (justify left))
     )
-    (property "Footprint" "zzkeeb:Hole_M2-spacer" (at 39.37 314.96 0)
+    (property "Footprint" "zzkeeb:Hole_M2" (at 39.37 314.96 0)
       (effects (font (size 1.27 1.27)) hide)
     )
@@
       (effects (font (size 1.27 1.27)) (justify left))
     )
-    (property "Footprint" "zzkeeb:Hole_M2-spacer" (at 381 303.53 0)
+    (property "Footprint" "zzkeeb:Hole_M2" (at 381 303.53 0)
       (effects (font (size 1.27 1.27)) hide)
     )
@@
       (effects (font (size 1.27 1.27)) (justify left))
     )
-    (property "Footprint" "zzkeeb:Hole_M2-spacer" (at 358.14 322.58 0)
+    (property "Footprint" "zzkeeb:Hole_M2" (at 358.14 322.58 0)
       (effects (font (size 1.27 1.27)) hide)
     )
@@
       (effects (font (size 1.27 1.27)) (justify left))
     )
-    (property "Footprint" "zzkeeb:Hole_M2-spacer" (at 358.14 303.53 0)
+    (property "Footprint" "zzkeeb:Hole_M2" (at 358.14 303.53 0)
       (effects (font (size 1.27 1.27)) hide)
     )
@@
       (effects (font (size 1.27 1.27)) (justify left))
     )
-    (property "Footprint" "zzkeeb:Hole_M2-spacer" (at 39.37 302.26 0)
+    (property "Footprint" "zzkeeb:Hole_M2" (at 39.37 302.26 0)
       (effects (font (size 1.27 1.27)) hide)
     )
@@
       (effects (font (size 1.27 1.27)) (justify left))
     )
-    (property "Footprint" "zzkeeb:Hole_M2-spacer" (at 334.01 303.53 0)
+    (property "Footprint" "zzkeeb:Hole_M2" (at 334.01 303.53 0)
       (effects (font (size 1.27 1.27)) hide)
     )
@@
       (effects (font (size 1.27 1.27)) (justify left))
     )
-    (property "Footprint" "zzkeeb:Hole_M2-spacer" (at 39.37 308.61 0)
+    (property "Footprint" "zzkeeb:Hole_M2" (at 39.37 308.61 0)
       (effects (font (size 1.27 1.27)) hide)
     )
@@
       (effects (font (size 1.27 1.27)) (justify left))
     )
-    (property "Footprint" "zzkeeb:Hole_M2-spacer" (at 334.01 309.88 0)
+    (property "Footprint" "zzkeeb:Hole_M2" (at 334.01 309.88 0)
       (effects (font (size 1.27 1.27)) hide)
     )
@@
       (effects (font (size 1.27 1.27)) (justify left))
     )
-    (property "Footprint" "zzkeeb:Hole_M2-spacer" (at 64.77 314.96 0)
+    (property "Footprint" "zzkeeb:Hole_M2" (at 64.77 314.96 0)
       (effects (font (size 1.27 1.27)) hide)
     )
@@
       (effects (font (size 1.27 1.27)) (justify left))
     )
-    (property "Footprint" "zzkeeb:Hole_M2-spacer" (at 39.37 321.31 0)
+    (property "Footprint" "zzkeeb:Hole_M2" (at 39.37 321.31 0)
       (effects (font (size 1.27 1.27)) hide)
     )
@@
       (effects (font (size 1.27 1.27)) (justify left))
     )
-    (property "Footprint" "zzkeeb:Hole_M2-spacer" (at 64.77 302.26 0)
+    (property "Footprint" "zzkeeb:Hole_M2" (at 64.77 302.26 0)
       (effects (font (size 1.27 1.27)) hide)
     )
@@
       (effects (font (size 1.27 1.27)) (justify left))
     )
-    (property "Footprint" "zzkeeb:Hole_M2-spacer" (at 358.14 316.23 0)
+    (property "Footprint" "zzkeeb:Hole_M2" (at 358.14 316.23 0)
       (effects (font (size 1.27 1.27)) hide)
     )
@@
       (effects (font (size 1.27 1.27)) (justify left))
     )
-    (property "Footprint" "zzkeeb:Hole_M2-spacer" (at 64.77 308.61 0)
+    (property "Footprint" "zzkeeb:Hole_M2" (at 64.77 308.61 0)
       (effects (font (size 1.27 1.27)) hide)
     )
@@
       (effects (font (size 1.27 1.27)) (justify left))
     )
-    (property "Footprint" "zzkeeb:Hole_M2-spacer" (at 334.01 316.23 0)
+    (property "Footprint" "zzkeeb:Hole_M2" (at 334.01 316.23 0)
       (effects (font (size 1.27 1.27)) hide)
     )
@@
       (effects (font (size 1.27 1.27)) (justify left))
     )
-    (property "Footprint" "zzkeeb:Hole_M2-spacer" (at 64.77 321.31 0)
+    (property "Footprint" "zzkeeb:Hole_M2" (at 64.77 321.31 0)
       (effects (font (size 1.27 1.27)) hide)
     )
@@
       (effects (font (size 1.27 1.27)) (justify left))
     )
-    (property "Footprint" "zzkeeb:Hole_M2-spacer" (at 334.01 322.58 0)
+    (property "Footprint" "zzkeeb:Hole_M2" (at 334.01 322.58 0)
       (effects (font (size 1.27 1.27)) hide)
     )
@@
       (effects (font (size 1.27 1.27)) (justify left))
     )
-    (property "Footprint" "zzkeeb:Hole_M2-spacer" (at 358.14 309.88 0)
+    (property "Footprint" "zzkeeb:Hole_M2" (at 358.14 309.88 0)
       (effects (font (size 1.27 1.27)) hide)
     )
@@
       (effects (font (size 1.27 1.27)) (justify left))
     )
-    (property "Footprint" "zzkeeb:Hole_M2-spacer" (at 87.63 302.26 0)
+    (property "Footprint" "zzkeeb:Hole_M2" (at 87.63 302.26 0)
       (effects (font (size 1.27 1.27)) hide)
     )

Commit message: new jumper for VIK
Parts:
- added JP7, JP8: SolderJumper_3_Open, Jumper:SolderJumper-3_P1.3mm_Open_RoundedPad1.0x1.5mm, symbol Jumper:SolderJumper_3_Open
Connections:
- net BL: now also JP7.3 (B)
- net BL_r: now also JP8.3 (B)
- net GND: now also JP7.1 (A); no longer VIK_K1.7 (GND), VIK_K2.7 (GND), VIK_K3.7 (GND)
- net GNDA: now also JP8.1 (A); no longer VIK_K4.7 (GND), VIK_K5.7 (GND), VIK_K6.7 (GND)
- new net GND/BL: JP7.2 (C), VIK_K1.7 (GND), VIK_K2.7 (GND), VIK_K3.7 (GND)
- new net GND/BL_r: JP8.2 (C), VIK_K4.7 (GND), VIK_K5.7 (GND), VIK_K6.7 (GND)
Other:
- moved on the sheet: JP2, JP5, JP6

Commit message: final pcb
Parts:
- removed JP7, JP8: SolderJumper_3_Open, Jumper:SolderJumper-3_P1.3mm_Open_RoundedPad1.0x1.5mm, symbol Jumper:SolderJumper_3_Open
- VIK_K1, VIK_K4: footprint zzkeeb:Connector_VIK-vertical-keyboard -> vik:vik-keyboard-connector-vertical; symbol zzkeeb:Connector_VIK-keyboard -> vik:vik-keyboard-connector
- VIK_K2, VIK_K5: footprint zzkeeb:Connector_VIK-adapter-keyboard -> vik:vik-keyboard-throughole; symbol zzkeeb:Connector_VIK-keyboard -> vik:vik-keyboard-connector
- VIK_K3, VIK_K6: footprint zzkeeb:Connector_VIK-horizontal-keyboard -> vik:vik-keyboard-connector-horizontal; symbol zzkeeb:Connector_VIK-keyboard -> vik:vik-keyboard-connector
Connections:
- net GND/BL is gone; now on net GPIO1: VIK_K1.7 (GPIO_AD1), VIK_K2.7 (GPIO_AD1), VIK_K3.7 (GPIO_AD1)
- net GND/BL_r is gone; now on net GPIO1_r: VIK_K4.7 (GPIO_AD1), VIK_K5.7 (GPIO_AD1), VIK_K6.7 (GPIO_AD1)
- net BL renamed GPIO1
- net BL_r renamed GPIO1_r
- net RST renamed GPIO2
- net RST_r renamed GPIO2_r

Commit message: update 38keys to kicad 8, small routing updates, update libs
Parts:
- MCU1, MCU2: footprint zzkeeb:MCU_rp2040-zero-tht-pads -> zzkeeb:MCU_rp2040-zero-tht
- VIK_K1, VIK_K4: footprint vik:vik-keyboard-connector-vertical -> zzkeeb:Connector_VIK-vertical-keyboard
